File: AAMB.kicad_pcb (KiCad board)
At the start: 2 copper layers, 160.3 x 50.4 mm, 88 parts, among them Q201 BC546, Q202 BC546, Q203 BC546, Q204 BD140, Q205 BD139, Q206 BD140, Q207 MJL21193, Q208 MJL21194, Q209 BC546, Q301 BC546, Q302 BC546, Q303 BC546, Q304 BD140, Q305 BD139, Q306 BD140, Q307 MJL21193, Q308 MJL21194, Q309 BC546

Commit message: Testing branch. Pulled parts into layout.
Parts:
- removed JN351, JN352, JP351, JP352, J_IN_L1, J_IN_R1, J_OUT_L1, J_OUT_R1: Conn_01x02_Female, Connectors_Molex:Molex_KK-41791-02_02x3.96mm_Straight
- added C1: 10u, Capacitor_SMD:C_1206_3216Metric_Pad1.42x1.75mm_HandSolder, F.Cu at (19.0, 69.6)
- added C10: 1000u, Capacitor_SMD:C_Elec_10x10.2, F.Cu at (111.5, -15.2)
- added C11: 22p, Capacitor_SMD:C_0603_1608Metric_Pad1.05x0.95mm_HandSolder, F.Cu at (134.4, -22.8)
- added C12: 22p, Capacitor_SMD:C_0603_1608Metric_Pad1.05x0.95mm_HandSolder, F.Cu at (134.4, -25.3)
- added C13: 10u, Capacitor_THT:CP_Radial_D5.0mm_P2.00mm, F.Cu at (128.0, -23.3)
- added C14: 10u, Capacitor_THT:CP_Radial_D5.0mm_P2.00mm, F.Cu at (121.4, -23.3)
- added C15: 0.1u, Capacitor_SMD:C_0603_1608Metric_Pad1.05x0.95mm_HandSolder, F.Cu at (138.1, -29.2)
- added C16: 0.1u, Capacitor_SMD:C_0603_1608Metric_Pad1.05x0.95mm_HandSolder, F.Cu at (138.1, -31.8)
- added C17: 0.1u, Capacitor_SMD:C_0603_1608Metric_Pad1.05x0.95mm_HandSolder, F.Cu at (120.8, -7.19)
- added C18: 0.1u, Capacitor_SMD:C_0603_1608Metric_Pad1.05x0.95mm_HandSolder, F.Cu at (138.8, -24.2)
- added C19: 0.1u, Capacitor_SMD:C_0603_1608Metric_Pad1.05x0.95mm_HandSolder, F.Cu at (125.5, -9.70)
- added C2: 10u, Capacitor_SMD:C_1206_3216Metric_Pad1.42x1.75mm_HandSolder, B.Cu at (234.4, 84.1)
- added C20: 0.1u, Capacitor_SMD:C_0603_1608Metric_Pad1.05x0.95mm_HandSolder, F.Cu at (127.8, -18.8)
- added C21: 0.1u, Capacitor_SMD:C_0603_1608Metric_Pad1.05x0.95mm_HandSolder, F.Cu at (136.5, -20.3)
- added C22: 0.1u, Capacitor_SMD:C_0603_1608Metric_Pad1.05x0.95mm_HandSolder, F.Cu at (121.2, -12.2)
- added C23: 0.1u, Capacitor_SMD:C_0603_1608Metric_Pad1.05x0.95mm_HandSolder, F.Cu at (72.8, 34.2)
- added C24: 0.1u, Capacitor_SMD:C_0603_1608Metric_Pad1.05x0.95mm_HandSolder, F.Cu at (63.8, 40.9)
- added C3: 10u, Capacitor_THT:CP_Radial_D5.0mm_P2.00mm, F.Cu at (28.5, 57.5)
- added C4: 1u, Capacitor_THT:CP_Radial_D5.0mm_P2.00mm, F.Cu at (22.6, 64.7)
- added C5: 10u, Capacitor_SMD:C_1206_3216Metric_Pad1.42x1.75mm_HandSolder, F.Cu at (29.9, 62.4)
- added C6: 10u, Capacitor_SMD:C_1206_3216Metric_Pad1.42x1.75mm_HandSolder, F.Cu at (46.4, 44.9)
- added C7: 10u, Capacitor_THT:CP_Radial_D5.0mm_P2.00mm, F.Cu at (114.4, -6.04)
- added C8: 10u, Capacitor_THT:CP_Radial_D5.0mm_P2.00mm, F.Cu at (121.4, -16.7)
- added C9: 1000u, Capacitor_SMD:C_Elec_10x10.2, F.Cu at (111.5, -27.1)
- added D1: 1N4004, Diode_THT:D_DO-41_SOD81_P10.16mm_Horizontal, F.Cu at (29.3, 39.3)
- added D10: 1N4004, Diode_THT:D_DO-41_SOD81_P10.16mm_Horizontal, F.Cu at (15.4, 47.8)
- added D11: 24V, Diode_SMD:D_SMA, F.Cu at (16.2, 63.7)
- added D12: 1N4004, Diode_THT:D_DO-41_SOD81_P10.16mm_Horizontal, F.Cu at (29.3, 43.6)
- added D13: 24V, Diode_SMD:D_SMA, F.Cu at (45.3, 35.2)
- added D2: 1N4004, Diode_THT:D_DO-41_SOD81_P10.16mm_Horizontal, F.Cu at (15.4, 52.1)
- added D3: 1N4004, Diode_THT:D_DO-41_SOD81_P10.16mm_Horizontal, F.Cu at (15.4, 39.3)
- added D4: 1N4004, Diode_THT:D_DO-41_SOD81_P10.16mm_Horizontal, F.Cu at (14.1, 59.3)
- added D5: 1N4004, Diode_THT:D_DO-41_SOD81_P10.16mm_Horizontal, F.Cu at (-20.7, 69.8)
- added D6: 1N4004, Diode_THT:D_DO-41_SOD81_P10.16mm_Horizontal, F.Cu at (15.4, 35.1)
- added D7: 1N4004, Diode_THT:D_DO-41_SOD81_P10.16mm_Horizontal, F.Cu at (-6.81, 69.8)
- added D8: 1N4004, Diode_THT:D_DO-41_SOD81_P10.16mm_Horizontal, F.Cu at (15.4, 43.6)
- added D9: 1N4004, Diode_THT:D_DO-41_SOD81_P10.16mm_Horizontal, F.Cu at (29.3, 35.1)
- added J1: Screw_Terminal_01x04, TerminalBlock_Phoenix:TerminalBlock_Phoenix_MKDS-1,5-4_1x04_P5.00mm_Horizontal, F.Cu at (168.1, 77.5)
- added J2: PJRAS4X2U01X, Connectors-amp:PJRAS4X2U01X, F.Cu at (-4.95, -4.06)
- added J3: SPKR L, TerminalBlock_Phoenix:TerminalBlock_Phoenix_MKDS-1,5-2_1x02_P5.00mm_Horizontal, F.Cu at (48.2, -26.8)
- added J4: SPKR R, TerminalBlock_Phoenix:TerminalBlock_Phoenix_MKDS-1,5-2_1x02_P5.00mm_Horizontal, F.Cu at (4.08, -3.06)
- added J5: Screw_Terminal_01x03, TerminalBlock_Phoenix:TerminalBlock_Phoenix_MKDS-1,5-3_1x03_P5.00mm_Horizontal, F.Cu at (21.1, -14.9)
- added J6: Screw_Terminal_01x03, TerminalBlock_Phoenix:TerminalBlock_Phoenix_MKDS-1,5-3_1x03_P5.00mm_Horizontal, F.Cu at (4.08, -14.9)
- added J7: Screw_Terminal_01x04, TerminalBlock_Phoenix:TerminalBlock_Phoenix_MKDS-1,5-4_1x04_P5.00mm_Horizontal, F.Cu at (4.08, -26.8)
- added K1: G5LE-1, Relay_THT:Relay_SPDT_Omron-G5LE-1, F.Cu at (-13.6, 36.4)
- added K2: G5LE-1, Relay_THT:Relay_SPDT_Omron-G5LE-1, F.Cu at (4.48, 36.4)
- added Q1: BC546, Package_TO_SOT_THT:TO-92_Inline, F.Cu at (43.3, 40.7)
- added Q2: BC556, Package_TO_SOT_THT:TO-92_Inline, F.Cu at (38.9, 48.9)
- added Q3: BC546, Package_TO_SOT_THT:TO-92_Inline, F.Cu at (34.7, 54.7)
- added Q4: BD140, Package_TO_SOT_THT:TO-126-3_Vertical, F.Cu at (29.6, 48.5)
- added R1: 100k, Resistor_SMD:R_0603_1608Metric_Pad1.05x0.95mm_HandSolder, F.Cu at (29.1, 65.3)
- added R10: 10k, Resistor_SMD:R_0603_1608Metric_Pad1.05x0.95mm_HandSolder, F.Cu at (24.1, 71.7)
- added R11: 10k, Resistor_SMD:R_0603_1608Metric_Pad1.05x0.95mm_HandSolder, F.Cu at (41.4, 55.2)
- added R12: 100k, Resistor_SMD:R_0603_1608Metric_Pad1.05x0.95mm_HandSolder, F.Cu at (29.1, 67.8)
- added R13: 150, Resistor_THT:R_Axial_DIN0207_L6.3mm_D2.5mm_P7.62mm_Horizontal, F.Cu at (6.80, 69.7)
- added R14: 3.9, Resistor_THT:R_Axial_Power_L25.0mm_W9.0mm_P10.16mm_Vertical, F.Cu at (0.09, 62.4)
- added R15: 3.9, Resistor_THT:R_Axial_Power_L25.0mm_W9.0mm_P10.16mm_Vertical, F.Cu at (-17.3, 62.4)
- added R16: 1k5, Resistor_SMD:R_0603_1608Metric_Pad1.05x0.95mm_HandSolder, F.Cu at (121.2, -9.70)
- added R17: 1k5, Resistor_SMD:R_0603_1608Metric_Pad1.05x0.95mm_HandSolder, F.Cu at (127.8, -16.2)
- added R18: 2k2, Resistor_SMD:R_0603_1608Metric_Pad1.05x0.95mm_HandSolder, F.Cu at (142.4, -31.8)
- added R19: 1M, Resistor_SMD:R_0603_1608Metric_Pad1.05x0.95mm_HandSolder, F.Cu at (132.2, -18.8)
- added R2: 100k, Resistor_SMD:R_0603_1608Metric_Pad1.05x0.95mm_HandSolder, B.Cu at (229.1, 82.5)
- added R20: 100, Resistor_SMD:R_0603_1608Metric_Pad1.05x0.95mm_HandSolder, F.Cu at (142.4, -29.2)
- added R21: 100, Resistor_SMD:R_0603_1608Metric_Pad1.05x0.95mm_HandSolder, F.Cu at (138.8, -26.7)
- added R22: 22k, Resistor_SMD:R_0603_1608Metric_Pad1.05x0.95mm_HandSolder, F.Cu at (125.5, -12.2)
- added R23: 22k, Resistor_SMD:R_0603_1608Metric_Pad1.05x0.95mm_HandSolder, F.Cu at (125.2, -4.68)
- added R24: 38.3k, Resistor_SMD:R_0603_1608Metric_Pad1.05x0.95mm_HandSolder, F.Cu at (72.5, 40.9)
- added R25: 2k2, Resistor_SMD:R_0603_1608Metric_Pad1.05x0.95mm_HandSolder, F.Cu at (132.2, -16.2)
- added R26: 22k, Resistor_SMD:R_0603_1608Metric_Pad1.05x0.95mm_HandSolder, F.Cu at (129.5, -7.19)
- added R27: 22k, Resistor_SMD:R_0603_1608Metric_Pad1.05x0.95mm_HandSolder, F.Cu at (134.2, -13.7)
- added R28: 100, Resistor_SMD:R_0603_1608Metric_Pad1.05x0.95mm_HandSolder, F.Cu at (140.9, -21.7)
- added R29: 100, Resistor_SMD:R_0603_1608Metric_Pad1.05x0.95mm_HandSolder, F.Cu at (136.5, -17.8)
- added R3: 10, Resistor_SMD:R_0603_1608Metric_Pad1.05x0.95mm_HandSolder, F.Cu at (41.4, 52.7)
- added R30: 5k1, Resistor_SMD:R_0603_1608Metric_Pad1.05x0.95mm_HandSolder, F.Cu at (129.9, -11.2)
- added R31: 5k1, Resistor_SMD:R_0603_1608Metric_Pad1.05x0.95mm_HandSolder, F.Cu at (143.1, -24.2)
- added R32: 22k, Resistor_SMD:R_0603_1608Metric_Pad1.05x0.95mm_HandSolder, F.Cu at (125.2, -7.19)
- added R33: 22k, Resistor_SMD:R_0603_1608Metric_Pad1.05x0.95mm_HandSolder, F.Cu at (129.9, -13.7)
- added R34: 100, Resistor_SMD:R_0603_1608Metric_Pad1.05x0.95mm_HandSolder, F.Cu at (143.1, -26.7)
- added R35: 100, Resistor_SMD:R_0603_1608Metric_Pad1.05x0.95mm_HandSolder, F.Cu at (120.8, -4.68)
- added R36: 10k, Resistor_SMD:R_0603_1608Metric_Pad1.05x0.95mm_HandSolder, F.Cu at (68.2, 43.5)
- added R37: 2k2, Resistor_SMD:R_0603_1608Metric_Pad1.05x0.95mm_HandSolder, F.Cu at (72.8, 36.7)
- added R38: 22k, Resistor_SMD:R_0603_1608Metric_Pad1.05x0.95mm_HandSolder, F.Cu at (68.2, 40.9)
- added R39: 22k, Resistor_SMD:R_0603_1608Metric_Pad1.05x0.95mm_HandSolder, F.Cu at (63.8, 43.5)
- added R4: 100k, Resistor_SMD:R_0603_1608Metric_Pad1.05x0.95mm_HandSolder, F.Cu at (24.1, 69.2)
- added R5: 22k, Resistor_SMD:R_0603_1608Metric_Pad1.05x0.95mm_HandSolder, F.Cu at (18.2, 72.5)
- added R6: 22k, Resistor_SMD:R_0603_1608Metric_Pad1.05x0.95mm_HandSolder, F.Cu at (29.6, 51.7)
- added R7: 100k, Resistor_SMD:R_0603_1608Metric_Pad1.05x0.95mm_HandSolder, F.Cu at (15.7, 55.4)
- added R8: 100k, Resistor_SMD:R_0603_1608Metric_Pad1.05x0.95mm_HandSolder, F.Cu at (35.0, 61.8)
- added R9: 10k, Resistor_SMD:R_0603_1608Metric_Pad1.05x0.95mm_HandSolder, F.Cu at (20.0, 55.4)
- added TP1: post_sw_pre_vol_L, TestPoint:TestPoint_2Pads_Pitch2.54mm_Drill0.8mm, F.Cu at (14.6, -7.27)
- added TP2: post_sw_pre_vol_R, TestPoint:TestPoint_2Pads_Pitch2.54mm_Drill0.8mm, F.Cu at (2.58, 4.59)
- added TP3: post_vol_pre_amp_L, TestPoint:TestPoint_2Pads_Pitch2.54mm_Drill0.8mm, F.Cu at (2.58, 8.64)
- added TP4: post_vol_pre_amp_R, TestPoint:TestPoint_2Pads_Pitch2.54mm_Drill0.8mm, F.Cu at (14.6, -3.22)
- added TP5: post_amp_pre_rly_L, TestPoint:TestPoint_2Pads_Pitch2.54mm_Drill0.8mm, F.Cu at (36.7, -19.1)
- added TP6: post_amp_pre_rly_R, TestPoint:TestPoint_2Pads_Pitch2.54mm_Drill0.8mm, F.Cu at (-20.6, 26.9)
- added U1: TL072, Package_SO:SOIC-8_3.9x4.9mm_P1.27mm, F.Cu at (107.8, -6.09)
- added U2: NE5532, Package_SO:SOIC-8_3.9x4.9mm_P1.27mm, F.Cu at (131.7, -29.8)
- added U3: NE5532, Package_SO:SOIC-8_3.9x4.9mm_P1.27mm, F.Cu at (123.2, -29.8)
- added U4: THAT2180, Package_DIP:DIP-16_W7.62mm_SMDSocket_SmallPads, F.Cu at (98.2, -22.0)
- added U5: DG509BEQ-T1-E3, Package_SO:TSSOP-16_4.4x5mm_P0.65mm, F.Cu at (66.1, 36.4)
- added U6: CD4071B, Package_SO:SOIC-14_3.9x8.7mm_P1.27mm, F.Cu at (57.4, 38.0)
- added VR1: 5k, Murata-POT:PV36W202C01B00, F.Cu at (100.4, -7.64)
- R205: moved to F.Cu
- moved C307 7.90 mm to (232.9, 80.3), turned to 0 degrees
- moved R315 5.40 mm to (229.1, 80.3)
- moved R215 5.29 mm to (151.6, 80.3)
- moved R205 1.97 mm to (137.4, 80.3), turned to 0 degrees
Connections:
- net /audio_pwr_L/OUT_L renamed /pwr_audio_L
- net /audio_pwr_R/OUT_R renamed /pwr_audio_R
- C201 pad 1: /audio_pwr_L/IN_L -> /line_audio_L
- C301 pad 1: /audio_pwr_R/IN_R -> /line_audio_R
- F201 pad 1: /audio_pwr_L/P35 -> +35V
- F202 pad 1: /audio_pwr_L/N35 -> -35V
- F301 pad 1: /audio_pwr_R/P35 -> +35V
- F302 pad 1: /audio_pwr_R/N35 -> -35V
Routing:
- net -35V: track 0.00 -> 118.7 mm
- net +35V: track 0.00 -> 102.1 mm
- net Net-(C305-Pad2): track 44.7 -> 6.47 mm, vias 1 -> 0
- net Net-(C205-Pad2): track 41.8 -> 6.49 mm, vias 1 -> 0
- net /audio_pwr_R/N35: track 18.8 -> 0.00 mm
- net /audio_pwr_L/N35: track 17.8 -> 0.00 mm
- net /audio_pwr_L/IN_L: track 15.4 -> 0.00 mm
- net /audio_pwr_R/IN_R: track 13.9 -> 0.00 mm
- net /audio_pwr_L/P35: track 12.7 -> 0.00 mm
- net /audio_pwr_R/P35: track 12.3 -> 0.00 mm
- net /pwr_audio_L: track 33.2 -> 28.9 mm
- net Net-(C2-Pad1): track 0.00 -> 3.60 mm
- net /pwr_audio_R: track 33.2 -> 29.7 mm
- net Net-(C307-Pad1): track 6.28 -> 2.94 mm
- net Net-(C207-Pad1): track 6.80 -> 9.44 mm
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Other:
- board size 160.3 x 50.4 mm -> 160.2 x 120.1 mm

Commit message: 23JAN2020 daily commit.
Parts:
- removed the R15 at (-17.3, 62.4)
- removed the R310 at (189.1, 48.9)
- added C6: 10u, Capacitor_SMD:C_1206_3216Metric_Pad1.42x1.75mm_HandSolder, F.Cu at (314.4, 14.3)
- added D2: 1N4004, Diode_THT:D_DO-41_SOD81_P10.16mm_Horizontal, F.Cu at (313.8, -4.57)
- C2, R2, R203, R204, R206, R207, R208, R209, R210, R212, R215, R303, R304, R305, R306, R307, R308, R309, R311, R312, R315: moved to F.Cu
- R15: renamed from C6; value 10u -> 3.9; footprint Capacitor_SMD:C_1206_3216Metric_Pad1.42x1.75mm_HandSolder -> Resistor_THT:R_Axial_Power_L25.0mm_W9.0mm_P10.16mm_Vertical
- R213, R214, R313, R314: footprint Resistor_THT:R_Axial_Power_L25.0mm_W9.0mm_P30.48mm -> Resistor_THT:R_Axial_Power_L25.0mm_W9.0mm_P10.16mm_Vertical
- R310: renamed from D2; value 1N4004 -> 3.3k; footprint Diode_THT:D_DO-41_SOD81_P10.16mm_Horizontal -> Resistor_SMD:R_0603_1608Metric_Pad1.05x0.95mm_HandSolder
- moved U2 376.2 mm to (-243.7, -5.46)
- moved R18 369.6 mm to (-226.3, -6.56)
- moved R20 368.8 mm to (-226.0, -11.6)
- moved R27 364.6 mm to (-230.3, -9.07)
- moved R25 363.0 mm to (-230.7, -4.05)
- moved R34 362.6 mm to (-219.3, -15.6)
- moved C21 360.2 mm to (-223.7, -18.1)
- moved R30 360.2 mm to (-230.3, -11.6)
- moved R28 357.9 mm to (-217.1, -22.2)
- moved R31 356.6 mm to (-213.4, -28.6)
- moved C12 356.4 mm to (-221.6, -10.6)
- moved C18 356.2 mm to (-217.3, -13.1)
- moved R33 355.9 mm to (-226.0, -9.07)
- moved R29 353.6 mm to (-217.1, -24.7)
- moved R26 353.3 mm to (-223.7, -15.6)
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Connections:
- R15 pad 1: Net-(C6-Pad1) -> Net-(C5-Pad1)
- R15 pad 2: /short_protection_muting/audio_rly_out_L -> /pwr_audio_R
- R214 pad 1: /pwr_audio_L -> /audio_pwr_L/pwr_fet_neg_L
- R214 pad 2: /audio_pwr_L/pwr_fet_neg_L -> /pwr_audio_L
- R310 pad 1: Net-(D1-Pad1) -> Net-(C305-Pad2)
- R310 pad 2: Net-(C2-Pad1) -> /audio_pwr_R/N35_fused_R
- R314 pad 1: /pwr_audio_R -> /audio_pwr_R/pwr_fet_neg_R
- R314 pad 2: /audio_pwr_R/pwr_fet_neg_R -> /pwr_audio_R
Routing:
- net /audio_pwr_R/P35_fused_R: track 65.1 -> 12.1 mm
- net /audio_pwr_L/P35_fused_L: track 68.1 -> 18.3 mm
- net /audio_pwr_R/N35_fused_R: track 60.7 -> 12.7 mm
- net Net-(Q201-Pad3): track 46.4 -> 0.00 mm
- net Net-(Q301-Pad3): track 46.1 -> 0.00 mm
- net Net-(C204-Pad2): track 45.9 -> 0.00 mm
- net Net-(C304-Pad2): track 44.0 -> 0.00 mm
- net -35V: track 118.7 -> 75.8 mm
- net Net-(C206-Pad2): track 42.4 -> 0.00 mm
- net Net-(Q202-Pad2): track 30.0 -> 0.00 mm, vias 2 -> 0
- net Net-(Q302-Pad2): track 28.5 -> 0.00 mm, vias 1 -> 0
- net /audio_pwr_L/N35_fused_L: track 60.0 -> 32.3 mm
- net Net-(C206-Pad1): track 26.6 -> 0.00 mm, vias 1 -> 0
- net Net-(C306-Pad2): track 25.6 -> 0.00 mm
- net Net-(C306-Pad1): track 25.0 -> 0.00 mm
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- removed copper zone on B.Cu, net GND
- removed copper zone on F.Cu, net GND
Other:
- board outline removed
- net class audio_3A removed
- net class audio_5A added: clearance 0.5, trace_width 2, via_dia 2.6, via_drill 1.3

Commit message: 24JAN2020 daily
Parts:
- added R40: 0R, Resistor_SMD:R_2010_5025Metric_Pad1.52x2.65mm_HandSolder, F.Cu at (88.9, 51.7)
- added R41: 0R, Resistor_SMD:R_2010_5025Metric_Pad1.52x2.65mm_HandSolder, F.Cu at (119.3, 42.5)
- added R42: 0R, Resistor_SMD:R_2010_5025Metric_Pad1.52x2.65mm_HandSolder, F.Cu at (80.4, 42.4)
- added R43: 0R, Resistor_SMD:R_2010_5025Metric_Pad1.52x2.65mm_HandSolder, F.Cu at (152.9, 42.7)
- added R44: 0R, Resistor_SMD:R_2010_5025Metric_Pad1.52x2.65mm_HandSolder, F.Cu at (191.7, 44.3)
- added R45: 0R, Resistor_SMD:R_2010_5025Metric_Pad1.52x2.65mm_HandSolder, F.Cu at (159.8, 42.5)
- C1, C2, C5, C6, D11, D13, R1, R10, R11, R2, R202, R203, R204, R205, R206, R207, R208, R209, R210, R215, R216, R3, R305, R307, R308, R309, R310, R311, R312, R4, R5, R6, R7, R8, R9: moved to B.Cu
- moved Q3 314.3 mm to (19.2, 79.5)
- moved R4 302.1 mm to (31.5, 45.4), turned to 90 degrees
- moved R3 299.0 mm to (29.7, 45.4), turned to 90 degrees
- moved Q2 298.3 mm to (30.9, 82.9), turned to 270 degrees
- moved R12 297.7 mm to (22.0, 60.8), turned to 270 degrees
- moved C4 297.5 mm to (22.5, 73.6)
- moved R9 294.0 mm to (20.5, 82.0)
- moved R8 293.4 mm to (35.1, 45.4), turned to 270 degrees
- moved R10 293.0 mm to (20.0, 77.2)
- moved D8 292.9 mm to (18.9, 73.9), turned to 90 degrees
- moved Q4 289.6 mm to (37.7, 86.6), turned to 90 degrees
- moved R7 281.5 mm to (33.3, 45.4), turned to 90 degrees
- moved C3 277.3 mm to (32.0, 51.0)
- moved D9 272.3 mm to (42.3, 88.0), turned to 90 degrees
- moved R5 271.5 mm to (48.8, 77.1), turned to 90 degrees
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Connections:
- C205 pad 1: /pwr_audio_L -> Net-(C205-Pad1)
- C305 pad 1: /pwr_audio_R -> Net-(C305-Pad1)
- D201 pad 1: /audio_pwr_L/N35_fused_L -> /audio_pwr_L/N35_low_pow_L
- D301 pad 1: /audio_pwr_R/N35_fused_R -> /audio_pwr_R/N35_low_pow_R
- Q202 pad 1: /audio_pwr_L/P35_fused_L -> /audio_pwr_L/P35_low_pow_L
- Q204 pad 1: /audio_pwr_L/P35_fused_L -> /audio_pwr_L/P35_low_pow_L
- Q302 pad 1: /audio_pwr_R/P35_fused_R -> /audio_pwr_R/P35_low_pow_R
- Q304 pad 1: /audio_pwr_R/P35_fused_R -> /audio_pwr_R/P35_low_pow_R
- R205 pad 1: /pwr_audio_L -> Net-(C205-Pad1)
- R206 pad 1: /audio_pwr_L/P35_fused_L -> /audio_pwr_L/P35_low_pow_L
- R207 pad 2: /audio_pwr_L/N35_fused_L -> /audio_pwr_L/N35_low_pow_L
- R210 pad 2: /audio_pwr_L/N35_fused_L -> /audio_pwr_L/N35_low_pow_L
- R211 pad 2: /audio_pwr_L/N35_fused_L -> /audio_pwr_L/N35_low_pow_L
- R212 pad 1: /audio_pwr_L/P35_fused_L -> /audio_pwr_L/P35_low_pow_L
- R305 pad 1: /pwr_audio_R -> Net-(C305-Pad1)
- R306 pad 1: /audio_pwr_R/P35_fused_R -> /audio_pwr_R/P35_low_pow_R
- R307 pad 2: /audio_pwr_R/N35_fused_R -> /audio_pwr_R/N35_low_pow_R
- R310 pad 2: /audio_pwr_R/N35_fused_R -> /audio_pwr_R/N35_low_pow_R
- R311 pad 2: /audio_pwr_R/N35_fused_R -> /audio_pwr_R/N35_low_pow_R
- R312 pad 1: /audio_pwr_R/P35_fused_R -> /audio_pwr_R/P35_low_pow_R
Routing:
- net +35V: track 108.0 -> 0.00 mm
- net -35V: track 75.8 -> 0.00 mm
- net /audio_pwr_L/N35_fused_L: track 32.3 -> 0.00 mm
- net /pwr_audio_L: track 20.6 -> 0.00 mm
- net /pwr_audio_R: track 19.2 -> 0.00 mm
- net /audio_pwr_L/P35_fused_L: track 18.3 -> 0.00 mm
- net /audio_pwr_L/pwr_fet_pos_L: track 16.3 -> 0.00 mm
- net /audio_pwr_L/pwr_fet_neg_L: track 16.2 -> 0.00 mm
- net /audio_pwr_R/pwr_fet_neg_R: track 16.2 -> 0.00 mm
- net /audio_pwr_R/pwr_fet_pos_R: track 15.9 -> 29.0 mm
- net /audio_pwr_R/N35_fused_R: track 12.7 -> 0.00 mm
- net Net-(Q305-Pad2): track 0.00 -> 1.00 mm
- net Net-(Q205-Pad2): track 0.00 -> 1.00 mm
- added copper zone on B.Cu, net GND
- added copper zone on F.Cu, net GND

Commit message: Daily commit and ready to merge back to master.
Parts:
- moved R313 81.4 mm to (253.8, -0.28)
- moved VR301 73.3 mm to (200.2, 96.9)
- moved Q208 70.7 mm to (25.7, -19.0)
- moved C209 70.4 mm to (45.3, -20.9)
- moved TP6 68.3 mm to (205.2, 123.4)
- moved C308 66.3 mm to (209.7, -11.9), turned to 90 degrees
- moved J4 65.4 mm to (166.7, 147.3)
- moved J1 64.5 mm to (-21.0, 6.38)
- moved C305 63.2 mm to (202.9, 21.0)
- moved R305 61.1 mm to (197.9, 12.5)
- moved C310 60.6 mm to (218.9, 8.08), turned to 270 degrees
- moved R43 58.3 mm to (210.2, 32.0), turned to 180 degrees
- moved Q302 58.1 mm to (193.4, 7.09), turned to 270 degrees
- moved K2 56.1 mm to (180.5, 114.4)
- moved C5 54.1 mm to (162.6, 133.4)
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Routing:
- net /audio_pwr_R/pwr_fet_pos_R: track 29.0 -> 0.00 mm
- net /audio_pwr_R/P35_fused_R: track 12.1 -> 0.00 mm
- net Net-(Q305-Pad2): track 1.00 -> 0.00 mm

Commit message: 26JAN2020 nightly. Continued placement arangment.
Parts:
- R201, R304, R306, R315, R316, R43: moved to B.Cu
- R309, R310, R311, R4, R7, R8: moved to F.Cu
- moved J7 237.9 mm to (98.5, 229.8)
- moved C23 228.1 mm to (124.8, 242.3)
- moved R24 228.1 mm to (124.8, 239.7)
- moved R37 228.1 mm to (120.5, 239.7)
- moved R38 228.1 mm to (120.5, 242.3)
- moved U6 228.1 mm to (114.1, 236.8)
- moved C24 228.1 mm to (129.4, 235.5)
- moved J2 228.1 mm to (123.0, 254.7)
- moved R36 228.1 mm to (129.2, 239.7)
- moved U5 228.1 mm to (123.5, 234.0)
- moved R39 228.1 mm to (130.1, 231.4)
- moved TP2 212.1 mm to (107.3, 229.4)
- moved J5 203.5 mm to (90.5, 211.8), turned to 270 degrees
- moved J6 196.5 mm to (116.7, 189.9), turned to 180 degrees
- moved TP1 193.9 mm to (128.8, 185.9), turned to 180 degrees
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Routing:
- net Net-(D3-Pad2): track 0.00 -> 27.8 mm
- net Net-(D9-Pad1): track 0.00 -> 20.8 mm
- net Net-(D1-Pad1): track 0.00 -> 15.3 mm
- net Net-(C4-Pad1): track 0.00 -> 12.7 mm
- net Net-(Q2-Pad1): track 0.00 -> 11.6 mm
- net Net-(Q2-Pad3): track 0.00 -> 9.49 mm
- net Net-(Q1-Pad1): track 0.00 -> 8.60 mm
- net Net-(C3-Pad2): track 0.00 -> 8.04 mm
- net Net-(Q2-Pad2): track 0.00 -> 6.80 mm
- net Net-(C1-Pad1): track 0.00 -> 6.15 mm
- net Net-(C2-Pad1): track 0.00 -> 5.07 mm
- net Net-(Q3-Pad1): track 0.00 -> 2.70 mm
- net Net-(C3-Pad1): track 0.00 -> 2.69 mm
- net Net-(Q3-Pad2): track 0.00 -> 2.53 mm
- net Net-(Q205-Pad2): track 1.00 -> 0.00 mm

Commit message: Prep to merge.
Parts:
- R212, R40: moved to B.Cu
- moved Q204 170.5 mm to (-37.3, -10.5)
- moved C204 170.5 mm to (-29.9, -1.97), turned to 180 degrees
- moved R206 169.1 mm to (-33.5, -5.97)
- moved Q202 164.0 mm to (-34.7, 3.81)
- moved Q201 164.0 mm to (-30.6, 1.27)
- moved R212 158.4 mm to (-35.0, -12.4)
- moved C210 137.1 mm to (-23.1, -5.59)
- moved C208 119.1 mm to (-17.3, -20.8)
- moved F201 119.1 mm to (-14.0, 6.92)
- moved Q205 119.1 mm to (-32.5, -14.7)
- moved Q207 119.1 mm to (-34.9, -21.1)
- moved R41 117.5 mm to (-20.4, -12.8)
- moved C6 112.4 mm to (61.3, 11.9)
- moved J3 112.4 mm to (63.5, 15.4)
- moved R205 99.6 mm to (-40.1, 6.92)
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