File: audio_pwr_L.kicad_sch (KiCad schematic)
At the start: 39 parts, among them Q203 BC846, Q204 BCP53, Q205 BCP56, Q206 BCP53, Q207 MJL21193, Q208 MJL21194, Q209 BC846, U201 BC846BDW1T1G

Commit message: Minor layout updates.
Changed lines of the file:
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@@
   (symbol (lib_id "Device:R") (at 163.83 121.92 0) (unit 1)
     (in_bom yes) (on_board yes)
-    (property "Reference" "R211" (id 0) (at 165.862 121.92 90))
+    (property "Reference" "R211" (id 0) (at 161.925 121.92 90))
     (property "Value" "220" (id 1) (at 163.83 121.92 90))
     (property "Footprint" "Resistor_SMD:R_0201_0603Metric_Pad0.64x0.40mm_HandSolder" (id 2) (at 162.052 121.92 90)
@@
   (symbol (lib_id "Device:R") (at 169.545 127 270) (unit 1)
     (in_bom yes) (on_board yes)
-    (property "Reference" "R42" (id 0) (at 169.545 121.7422 90))
-    (property "Value" "0R" (id 1) (at 169.545 124.0536 90))
+    (property "Reference" "R42" (id 0) (at 169.545 125.095 90))
+    (property "Value" "0R" (id 1) (at 169.545 127 90))
     (property "Footprint" "Resistor_SMD:R_2010_5025Metric" (id 2) (at 169.545 125.222 90)
       (effects (font (size 1.27 1.27)) hide)
@@
   (symbol (lib_id "Device:R") (at 169.545 48.26 270) (unit 1)
     (in_bom yes) (on_board yes)
-    (property "Reference" "R41" (id 0) (at 169.545 43.0022 90))
-    (property "Value" "0R" (id 1) (at 169.545 45.3136 90))
+    (property "Reference" "R41" (id 0) (at 169.545 46.355 90))
+    (property "Value" "0R" (id 1) (at 169.545 48.26 90))
     (property "Footprint" "Resistor_SMD:R_2010_5025Metric" (id 2) (at 169.545 46.482 90)
       (effects (font (size 1.27 1.27)) hide)
@@
   (symbol (lib_id "Device:R") (at 168.91 92.71 270) (unit 1)
     (in_bom yes) (on_board yes)
-    (property "Reference" "R40" (id 0) (at 168.91 87.4522 90))
-    (property "Value" "0R" (id 1) (at 168.91 89.7636 90))
+    (property "Reference" "R40" (id 0) (at 168.91 90.805 90))
+    (property "Value" "0R" (id 1) (at 168.91 92.71 90))
     (property "Footprint" "Resistor_SMD:R_2010_5025Metric" (id 2) (at 168.91 90.932 90)
       (effects (font (size 1.27 1.27)) hide)
