File: audio_pwr_R.kicad_sch (KiCad schematic)
At the start: 39 parts, among them Q303 BC846, Q304 BCP53, Q305 BCP56, Q306 BCP53, Q307 MJL21193, Q308 MJL21194, Q309 BC846, U301 BC846BDW1T1G

Commit message: Minor layout updates.
Parts:
- Q304: value BCP53 -> (none); footprint TO_SOT_Packages_THT:TO-126_Vertical -> (none)
Other:
- moved on the sheet: C307
Changed lines of the file:
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@@
   (junction (at 138.43 116.84) (diameter 0) (color 0 0 0 0)
   )
+  (junction (at 186.69 111.76) (diameter 0) (color 0 0 0 0)
+  )
   (junction (at 175.26 127) (diameter 0) (color 0 0 0 0)
   )
@@
   (junction (at 83.82 96.52) (diameter 0) (color 0 0 0 0)
   )
+  (junction (at 97.79 110.49) (diameter 0) (color 0 0 0 0)
+  )
+  (junction (at 76.2 110.49) (diameter 0) (color 0 0 0 0)
+  )
+  (junction (at 138.43 77.47) (diameter 0) (color 0 0 0 0)
+  )
+  (junction (at 114.3 48.26) (diameter 0) (color 0 0 0 0)
+  )
+  (junction (at 138.43 66.04) (diameter 0) (color 0 0 0 0)
+  )
+  (junction (at 189.23 62.23) (diameter 0) (color 0 0 0 0)
+  )
+  (junction (at 175.26 48.26) (diameter 0) (color 0 0 0 0)
+  )
+  (junction (at 163.83 116.84) (diameter 0) (color 0 0 0 0)
+  )
+  (junction (at 175.26 72.39) (diameter 0) (color 0 0 0 0)
+  )
+  (junction (at 107.95 102.87) (diameter 0) (color 0 0 0 0)
+  )
+  (junction (at 147.32 92.71) (diameter 0) (color 0 0 0 0)
+  )
+  (junction (at 107.95 127) (diameter 0) (color 0 0 0 0)
+  )
   (junction (at 186.69 124.46) (diameter 0) (color 0 0 0 0)
   )
-  (junction (at 97.79 110.49) (diameter 0) (color 0 0 0 0)
-  )
-  (junction (at 76.2 110.49) (diameter 0) (color 0 0 0 0)
-  )
-  (junction (at 138.43 77.47) (diameter 0) (color 0 0 0 0)
-  )
-  (junction (at 114.3 48.26) (diameter 0) (color 0 0 0 0)
-  )
-  (junction (at 138.43 66.04) (diameter 0) (color 0 0 0 0)
-  )
-  (junction (at 189.23 62.23) (diameter 0) (color 0 0 0 0)
-  )
-  (junction (at 175.26 48.26) (diameter 0) (color 0 0 0 0)
-  )
-  (junction (at 163.83 116.84) (diameter 0) (color 0 0 0 0)
-  )
-  (junction (at 175.26 72.39) (diameter 0) (color 0 0 0 0)
-  )
-  (junction (at 107.95 102.87) (diameter 0) (color 0 0 0 0)
-  )
-  (junction (at 147.32 92.71) (diameter 0) (color 0 0 0 0)
-  )
-  (junction (at 107.95 127) (diameter 0) (color 0 0 0 0)
-  )
   (junction (at 163.83 127) (diameter 0) (color 0 0 0 0)
   )
@@
   (junction (at 83.82 110.49) (diameter 0) (color 0 0 0 0)
   )
-  (junction (at 186.69 123.19) (diameter 0) (color 0 0 0 0)
-  )
   (junction (at 163.83 48.26) (diameter 0) (color 0 0 0 0)
   )
@@
     (stroke (width 0) (type default) (color 0 0 0 0))
   )
-  (wire (pts (xy 186.69 110.49) (xy 186.69 114.3))
+  (wire (pts (xy 186.69 110.49) (xy 186.69 111.76))
     (stroke (width 0) (type default) (color 0 0 0 0))
   )
@@
     (stroke (width 0) (type default) (color 0 0 0 0))
   )
+  (wire (pts (xy 186.69 123.19) (xy 186.69 124.46))
+    (stroke (width 0) (type default) (color 0 0 0 0))
+  )
   (wire (pts (xy 163.83 72.39) (xy 175.26 72.39))
     (stroke (width 0) (type default) (color 0 0 0 0))
@@
     (stroke (width 0) (type default) (color 0 0 0 0))
   )
+  (wire (pts (xy 186.69 102.87) (xy 186.69 104.14))
+    (stroke (width 0) (type default) (color 0 0 0 0))
+  )
   (wire (pts (xy 95.25 110.49) (xy 97.79 110.49))
     (stroke (width 0) (type default) (color 0 0 0 0))
@@
     (stroke (width 0) (type default) (color 0 0 0 0))
   )
-  (wire (pts (xy 186.69 121.92) (xy 186.69 123.19))
-    (stroke (width 0) (type default) (color 0 0 0 0))
-  )
   (wire (pts (xy 175.26 48.26) (xy 185.42 48.26))
     (stroke (width 0) (type default) (color 0 0 0 0))
@@
     (stroke (width 0) (type default) (color 0 0 0 0))
   )
-  (wire (pts (xy 186.69 123.19) (xy 186.69 124.46))
-    (stroke (width 0) (type default) (color 0 0 0 0))
-  )
   (wire (pts (xy 175.26 48.26) (xy 175.26 54.61))
     (stroke (width 0) (type default) (color 0 0 0 0))
@@
   )
   (wire (pts (xy 193.04 52.07) (xy 185.42 52.07))
+    (stroke (width 0) (type default) (color 0 0 0 0))
+  )
+  (wire (pts (xy 186.69 111.76) (xy 186.69 114.3))
     (stroke (width 0) (type default) (color 0 0 0 0))
   )
@@
     (pin "2")
   )
-  (symbol (lib_id "Device:C") (at 186.69 106.68 0) (unit 1)
-    (in_bom yes) (on_board yes)
-    (property "Reference" "C307" (id 0) (at 187.325 104.14 0)
-      (effects (font (size 1.27 1.27)) (justify left))
-    )
-    (property "Value" "100n" (id 1) (at 187.325 109.22 0)
-      (effects (font (size 1.27 1.27)) (justify left))
-    )
-    (property "Footprint" "Capacitor_THT:C_Rect_L7.2mm_W4.5mm_P5.00mm_FKS2_FKP2_MKS2_MKP2" (id 2) (at 187.6552 110.49 0)
-      (effects (font (size 1.27 1.27)) hide)
-    )
-    (property "Datasheet" "~" (id 3) (at 186.69 106.68 0)
-      (effects (font (size 1.27 1.27)) hide)
-    )
-    (property "DigiKey" "https://www.digikey.com/product-detail/en/kemet/R82EC3100AA70K/399-19335-ND/9685239" (id 4) (at 186.69 106.68 0)
-      (effects (font (size 1.27 1.27)) hide)
-    )
-    (property "MFG" "KEMET" (id 5) (at 186.69 106.68 0)
-      (effects (font (size 1.27 1.27)) hide)
-    )
-    (property "MPN" "R82EC3100AA70K" (id 6) (at 186.69 106.68 0)
+  (symbol (lib_id "Device:C") (at 186.69 107.95 0) (unit 1)
+    (in_bom yes) (on_board yes)
+    (property "Reference" "C307" (id 0) (at 187.325 105.41 0)
+      (effects (font (size 1.27 1.27)) (justify left))
+    )
+    (property "Value" "100n" (id 1) (at 187.325 110.49 0)
+      (effects (font (size 1.27 1.27)) (justify left))
+    )
+    (property "Footprint" "Capacitor_THT:C_Rect_L7.2mm_W4.5mm_P5.00mm_FKS2_FKP2_MKS2_MKP2" (id 2) (at 187.6552 111.76 0)
+      (effects (font (size 1.27 1.27)) hide)
+    )
+    (property "Datasheet" "~" (id 3) (at 186.69 107.95 0)
+      (effects (font (size 1.27 1.27)) hide)
+    )
+    (property "DigiKey" "https://www.digikey.com/product-detail/en/kemet/R82EC3100AA70K/399-19335-ND/9685239" (id 4) (at 186.69 107.95 0)
+      (effects (font (size 1.27 1.27)) hide)
+    )
+    (property "MFG" "KEMET" (id 5) (at 186.69 107.95 0)
+      (effects (font (size 1.27 1.27)) hide)
+    )
+    (property "MPN" "R82EC3100AA70K" (id 6) (at 186.69 107.95 0)
       (effects (font (size 1.27 1.27)) hide)
     )
@@
       (effects (font (size 1.27 1.27)) (justify left))
     )
-    (property "Value" "BCP53" (id 1) (at 140.97 55.88 0)
-      (effects (font (size 1.27 1.27)) (justify left))
-    )
-    (property "Footprint" "TO_SOT_Packages_THT:TO-126_Vertical" (id 2) (at 140.97 53.975 0)
+    (property "Value" "" (id 1) (at 140.97 55.88 0)
+      (effects (font (size 1.27 1.27)) (justify left))
+    )
+    (property "Footprint" "" (id 2) (at 140.97 53.975 0)
       (effects (font (size 1.27 1.27) italic) (justify left) hide)
     )
@@
   (symbol (lib_id "Device:R") (at 169.545 127 270) (unit 1)
     (in_bom yes) (on_board yes)
-    (property "Reference" "R45" (id 0) (at 169.545 121.7422 90))
-    (property "Value" "0R" (id 1) (at 169.545 124.0536 90))
+    (property "Reference" "R45" (id 0) (at 169.545 125.095 90))
+    (property "Value" "0R" (id 1) (at 169.545 127 90))
     (property "Footprint" "Resistor_SMD:R_2010_5025Metric" (id 2) (at 169.545 125.222 90)
       (effects (font (size 1.27 1.27)) hide)
@@
   (symbol (lib_id "Device:R") (at 169.545 48.26 270) (unit 1)
     (in_bom yes) (on_board yes)
-    (property "Reference" "R44" (id 0) (at 169.545 43.0022 90))
-    (property "Value" "0R" (id 1) (at 169.545 45.3136 90))
+    (property "Reference" "R44" (id 0) (at 169.545 46.355 90))
+    (property "Value" "0R" (id 1) (at 169.545 48.26 90))
     (property "Footprint" "Resistor_SMD:R_2010_5025Metric" (id 2) (at 169.545 46.482 90)
       (effects (font (size 1.27 1.27)) hide)
@@
   (symbol (lib_id "Device:R") (at 168.275 92.71 270) (unit 1)
     (in_bom yes) (on_board yes)
-    (property "Reference" "R43" (id 0) (at 168.275 87.4522 90))
-    (property "Value" "0R" (id 1) (at 168.275 89.7636 90))
+    (property "Reference" "R43" (id 0) (at 168.275 90.805 90))
+    (property "Value" "0R" (id 1) (at 168.275 92.71 90))
     (property "Footprint" "Resistor_SMD:R_2010_5025Metric" (id 2) (at 168.275 90.932 90)
       (effects (font (size 1.27 1.27)) hide)

Commit message: Updating layout and various changes. Backup commit.
Parts:
- Q304: value (none) -> BCP53; footprint (none) -> TO_SOT_Packages_THT:TO-126_Vertical
Connections:
- net audio_fb_lowpow_R: now reaches C305.1, R305.1, R43.2
